File: modular-psu-pfc-1.2kW.kicad_pcb (KiCad board)
At the start: 2 copper layers, 160 x 100 mm, 128 parts, among them J1 BLADE250, J2 BLADE250, J3 B4B-XH-A, J4 BLADE250, J5 BLADE250, K1 16A, Q1 50N60, Q2 50N60, Q3 847, Q4 847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

Commit message: Schematic & PCB updated.
Parts:
- removed R37: 0, Resistor_SMD:R_0805_2012Metric
- added C28: 105, Capacitor_SMD:C_1210_3225Metric, B.Cu at (226.0, 121.0)
- added C29: C, Capacitor_SMD:C_1206_3216Metric, B.Cu at (105.5, 115.0)
- added C30: 470, Capacitor_THT:CP_Radial_D10.0mm_P5.00mm, F.Cu at (96.9, 123.5)
- added C31: C, Capacitor_SMD:C_0805_2012Metric, B.Cu at (119.5, 118.9)
- added C32: C, Capacitor_SMD:C_0805_2012Metric, B.Cu at (124.5, 118.9)
- added C33: C, Capacitor_SMD:C_0805_2012Metric, B.Cu at (96.5, 141.1)
- added C34: 1000, Capacitor_THT:CP_Radial_D10.0mm_P5.00mm, F.Cu at (93.5, 143.4)
- added C35: 106, Capacitor_SMD:C_1210_3225Metric, B.Cu at (105.0, 141.0)
- added D15: 3H100, Diode_SMD:D_SMB, B.Cu at (100.5, 139.0)
- added D4: D_Filled, Diode_SMD:D_SOD-123, B.Cu at (109.5, 122.0)
- added D6: 3H100, Diode_SMD:D_SMB, B.Cu at (101.5, 124.5)
- added F3: 400mA, Fuse:Fuse_1812_4532Metric, B.Cu at (229.0, 97.0)
- added J6: XH, Connector_JST:JST_XH_B6B-XH-AM_1x06_P2.50mm_Vertical, F.Cu at (116.2, 144.5)
- added JP2: blob, Jumper:SolderJumper-2_P1.3mm_Open_RoundedPad1.0x1.5mm, B.Cu at (133.0, 141.5)
- added JP3: blob, Jumper:SolderJumper-2_P1.3mm_Open_RoundedPad1.0x1.5mm, B.Cu at (133.0, 146.5)
- added L3: 10, HR_Parts:INDUCTOR_SMD_4x4, B.Cu at (97.5, 146.0)
- added R35: R, Resistor_SMD:R_0805_2012Metric, B.Cu at (109.0, 119.0)
- added R51: R, Resistor_SMD:R_1206_3216Metric, B.Cu at (108.5, 115.0)
- added R52: R, Resistor_SMD:R_0805_2012Metric, B.Cu at (122.0, 118.9)
- added R53: R, Resistor_SMD:R_0805_2012Metric, B.Cu at (119.5, 122.9)
- added R54: R, Resistor_SMD:R_0805_2012Metric, B.Cu at (122.0, 122.9)
- added R55: R, Resistor_SMD:R_0805_2012Metric, B.Cu at (124.5, 122.9)
- added R56: R, Resistor_SMD:R_0805_2012Metric, B.Cu at (96.5, 137.1)
- added TX1: EF20-10P-V, HR_Parts:TRANSFORMER-EF20-10P-V, F.Cu at (113.0, 132.0)
- added U4: LNK626DG, Package_SO:PowerIntegrations_SO-8C, B.Cu at (115.0, 120.9)
- added U6: TLP291, Package_SO:SOP-4_7.5x4.1mm_P2.54mm, B.Cu at (125.5, 146.5)
- added U7: TLP291, Package_SO:SOP-4_7.5x4.1mm_P2.54mm, B.Cu at (125.5, 141.5)
- F2: value 1A -> 400mA; footprint Fuse:Fuse_1210_3225Metric -> Fuse:Fuse_1812_4532Metric
- J3: footprint Connector_JST:JST_EH_B4B-EH-A_1x04_P2.50mm_Vertical -> Connector_JST:JST_XH_B4B-XH-AM_1x04_P2.50mm_Vertical
- moved F2 103.2 mm to (224.5, 97.0), turned to -90 degrees
- moved J1 24.1 mm to (97.5, 111.5), turned to -90 degrees
- moved J5 19.4 mm to (90.8, 111.5), turned to -90 degrees
- moved D7 9.72 mm to (136.0, 147.3), turned to 90 degrees
- moved J3 9.27 mm to (149.5, 146.8), turned to 180 degrees
- moved R41 7.87 mm to (136.0, 141.5)
- moved C14 7.10 mm to (117.5, 111.5), turned to 90 degrees
- moved R48 6.96 mm to (132.0, 133.0), turned to 180 degrees
- moved Q3 6.71 mm to (132.0, 136.5), turned to 180 degrees
- moved R33 5.00 mm to (136.0, 136.5), turned to -90 degrees
- moved C22 4.50 mm to (139.0, 139.5)
- moved D13 4.50 mm to (141.5, 139.5)
- moved H7 2.50 mm to (217.5, 55.0)
- moved K1 0.50 mm to (97.8, 102.2)
Connections:
- net /PFC booster/+400V renamed +400V
- D7 pad 1: /PFC booster/~{RUN} -> Net-(D7-K)
- F2 pad 1: +12Vaux -> Net-(F2-Pad1)
- F2 pad 2: Net-(J3-Pin_1) -> Net-(F2-Pad2)
- J3 pad 1: Net-(J3-Pin_1) -> GND1
- J3 pad 2: /PFC booster/~{RUN} -> /PFC booster/~{ENABLE}
- J3 pad 3: /PFC booster/~{ENABLE} -> /PFC booster/~{RUN}
- J3 pad 4: GND1 -> +12Vaux
- K1 pad A1: /PFC booster/SS -> +12Vaux
- K1 pad A2: +12Vaux -> /PFC booster/SS
- L4 pad 3: Net-(L4-Pad3) -> Net-(F2-Pad1)
- L5 pad 4: Net-(L4-Pad3) -> Net-(F2-Pad2)
Routing:
- net Net-(L4-Pad3): track 16.0 -> 0.00 mm
- net /PFC booster/~{ENABLE}: track 70.1 -> 85.8 mm, vias 1 -> 0
- net +400V: track 48.1 -> 62.9 mm, vias 0 -> 1
- net Net-(F2-Pad2): track 0.00 -> 14.4 mm
- net Net-(J6-Pin_4): track 0.00 -> 13.8 mm
- net +5V: track 0.00 -> 13.2 mm
- net Net-(D15-K): track 0.00 -> 12.7 mm
- net Net-(J6-Pin_3): track 0.00 -> 11.8 mm
- net Net-(F2-Pad1): track 0.00 -> 10.8 mm
- net Net-(U4-FB): track 0.00 -> 8.92 mm
- net Net-(D15-A): track 0.00 -> 8.77 mm
- net Net-(J6-Pin_2): track 0.00 -> 8.41 mm
- net Net-(U4-BP): track 0.00 -> 8.24 mm
- net Net-(C25-Pad2): track 2.53 -> 10.2 mm
- net +12Vaux: track 330.9 -> 338.3 mm, vias 11 -> 10
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- added copper zone on B.Cu, net GND
- added copper zone on F.Cu, net GND
Other:
- board text removed: "Affix information label here"
