File: modular-psu-pfc-1.2kW.kicad_sch (KiCad schematic)
At the start: 39 parts, among them J1 BLADE250, J2 BLADE250, J3 B4B-XH-A, J4 BLADE250, J5 BLADE250, K1 16A, U1 CAP300DG

Commit message: Schematic & PCB updated.
Parts:
- removed F2: 1A, Fuse:Fuse_1210_3225Metric, symbol Device:Polyfuse
- removed J1, J5: BLADE250, HR_Parts:CON-BLADE250-VERTICAL, symbol Connector_Generic:Conn_01x01
- removed R37: 0, Resistor_SMD:R_0805_2012Metric, symbol Device:R
- added J6: XH, Connector_JST:JST_XH_B6B-XH-AM_1x06_P2.50mm_Vertical, symbol Connector_Generic:Conn_01x06
- added JP2, JP3: blob, Jumper:SolderJumper-2_P1.3mm_Open_RoundedPad1.0x1.5mm, symbol Jumper:SolderJumper_2_Open
- added U6, U7: TLP291, Package_SO:SOP-4_7.5x4.1mm_P2.54mm, symbol Isolator:TLP291
- J3: footprint Connector_JST:JST_EH_B4B-EH-A_1x04_P2.50mm_Vertical -> Connector_JST:JST_XH_B4B-XH-AM_1x04_P2.50mm_Vertical
Connections:
- net +12Vaux: now also J3.4 (Pin_4), K1.A1; no longer K1.A2
- net GND1: now also J3.1 (Pin_1), JP2.1 (A), U7.3; no longer J3.4 (Pin_4)
- net PFC booster/SS: now also K1.A2; no longer K1.A1
- net PFC booster/~{ENABLE}: now also J3.2 (Pin_2), JP2.2 (B), U7.4; no longer J3.3 (Pin_3)
- net PFC booster/~{RUN}: now also J3.3 (Pin_3), JP3.1 (A), U6.2; no longer D7.1 (K), J3.2 (Pin_2)
- new net: J6.3 (Pin_3), U7.1
- new net: J6.4 (Pin_4), U7.2
- new net: D7.1 (K), JP3.2 (B), U6.1
- new net: J6.1 (Pin_1), U6.4
- new net: J6.2 (Pin_2), U6.3
- new net +5V: J6.5 (Pin_5)
- new net GND: J6.6 (Pin_6)
Other:
- added sheet Aux. PSU (auxpsu.kicad_sch)
- sheet PFC booster ports: added none; removed +400V
- note added: "JP2: Short for always enabled. JP3: Short when U6 is not used."
- moved on the sheet: D2, D7, J3, R41, R46, R47, U1
