File: pfcbooster.kicad_sch (KiCad schematic)
At the start: 89 parts, among them Q1 50N60, Q2 50N60, Q3 847, Q4 847, Q6 1N60, Q7 847, Q8 847, SW1 70, U2 UCC2817A, U3 ZXGD3004E6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

Commit message: Schematic & PCB updated.
Parts:
- added C28: 105, Capacitor_SMD:C_1210_3225Metric, symbol Device:C
- added F2, F3: 400mA, Fuse:Fuse_1812_4532Metric, symbol Device:Polyfuse
- added J1, J5: BLADE250, HR_Parts:CON-BLADE250-VERTICAL, symbol Connector_Generic:Conn_01x01
Connections:
- net +400V: now also J1.1 (Pin_1)
- net GND1: now also J5.1 (Pin_1)
- net at C25.1, D10.2 (A), D11.1 (K): now also C28.1
- net at L4.3: now also F2.1, F3.1; no longer L5.4
- net at C25.2, L5.3: now also C28.2
- new net: F2.2, F3.2, L5.4
Other:
- note added: "Note 1: DNP where auxiliary supply U4 is installed. These are only required in variants that are powered from the auxiliary windings of L4 and L5."
- moved on the sheet: C10, C11, C12, C13, C14, C15, C16, C17, C18, C19, C20, C21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
